Commit message: Added rb10 code, need to fix gazebo tf tree

File: rbpodo_description/robots/rb10_1300e.urdf.xacro (robot description, xacro)
@@ -3,4 +3,7 @@
   <xacro:include filename="$(find rbpodo_description)/robots/rb_6dof.xacro" />
   <xacro:include filename="$(find rbpodo_description)/robots/rb_6dof.ros2_control.xacro" />
+  <xacro:include filename="$(find rbpodo_description)/robots/rb10_gazebo_control.xacro" />
+  <!-- <xacro:property name="ros2_control_params" value="$(find rbpodo_description)/configs/rb10_controller.yaml" />
+  <xacro:ignition_ros2_control_plugin ros2_control_params:="${ros2_control_params}"> -->
   <xacro:arg name="prefix" default="" />
   <xacro:arg name="robot_ip" default="10.0.2.7"/>

File: rbpodo_description/robots/rb_6dof.xacro (robot description, xacro)
@@ -28,5 +28,5 @@
     </link>
   </xacro:macro>
-  <xacro:macro name="joint" params="name model_id:=^">
+  <xacro:macro name="joint" params="name model_id:=^ prefix=''">
     <xacro:property name="joints_props_file" value="$(find rbpodo_description)/robots/${model_id}/joint.yaml" />
     <xacro:property name="joints_props" value="${xacro.load_yaml(joints_props_file)}" />
@@ -35,6 +35,6 @@
     <joint name="${name}" type="revolute">
       <origin xyz="${props.origin.xyz}" rpy="${props.origin.rpy}" />
-      <parent link="${props.parent}" />
-      <child link="${props.child}" />
+      <parent link="${prefix}${props.parent}" />
+      <child link="${prefix}${props.child}" />
       <axis xyz="${props.axis.xyz}" />
       <xacro:property name="limit" value="${props.limit}" />
@@ -43,5 +43,11 @@
   </xacro:macro>
   <xacro:macro name="rb_6dof" params="model_id prefix='' tcp_name='tcp' tcp_xyz='0 0 0' tcp_rpy='0 0 0'">
-    <xacro:link name="${prefix}link0" has_inertial="false" />
+    <link name="world" />
+    <joint name="${prefix}world_joint" type="fixed">
+      <parent link="world" />
+      <child link="${prefix}link0" />
+      <origin xyz="0 0 0" rpy="0 0 0" />
+    </joint>
+    <xacro:link name="${prefix}link0" has_inertial="true" />
     <xacro:link name="${prefix}link1" />
     <xacro:link name="${prefix}link2" />
@@ -51,10 +57,66 @@
     <xacro:link name="${prefix}link6" />
     <link name="${prefix}${tcp_name}" />
-    <xacro:joint name="${prefix}base" />
-    <xacro:joint name="${prefix}shoulder" />
-    <xacro:joint name="${prefix}elbow" />
-    <xacro:joint name="${prefix}wrist1" />
-    <xacro:joint name="${prefix}wrist2" />
-    <xacro:joint name="${prefix}wrist3" />
+    <xacro:joint name="${prefix}base" prefix="${prefix}"/>
+    <xacro:joint name="${prefix}shoulder" prefix="${prefix}"/>
+    <xacro:joint name="${prefix}elbow" prefix="${prefix}"/>
+    <xacro:joint name="${prefix}wrist1" prefix="${prefix}"/>
+    <xacro:joint name="${prefix}wrist2" prefix="${prefix}"/>
+    <xacro:joint name="${prefix}wrist3" prefix="${prefix}"/>
+    <!-- <xacro:property name="joints_props_file" value="$(find rbpodo_description)/robots/${model_id}/joint.yaml" />
+    <xacro:property name="joints_props" value="${xacro.load_yaml(joints_props_file)}" />
+    <xacro:property name="props" value="${joints_props['base']}" />
+    <joint name="${prefix}base" type="revolute">
+      <origin xyz="${props.origin.xyz}" rpy="${props.origin.rpy}" />
+      <parent link="${prefix}link0" />
+      <child link="${prefix}link1" />
+      <axis xyz="${props.axis.xyz}" />
+      <xacro:property name="limit" value="${props.limit}" />
+      <limit lower="${limit.lower}" upper="${limit.upper}" effort="${limit.effort}" velocity="${limit.velocity}" />
+    </joint>
+    <xacro:property name="props" value="${joints_props['shoulder']}" />
+    <joint name="${prefix}shoulder" type="revolute">
+      <origin xyz="${props.origin.xyz}" rpy="${props.origin.rpy}" />
+      <parent link="${prefix}link1" />
+      <child link="${prefix}link2" />
+      <axis xyz="${props.axis.xyz}" />
+      <xacro:property name="limit" value="${props.limit}" />
+      <limit lower="${limit.lower}" upper="${limit.upper}" effort="${limit.effort}" velocity="${limit.velocity}" />
+    </joint>
+    <xacro:property name="props" value="${joints_props['elbow']}" />
+    <joint name="${prefix}elbow" type="revolute">
+      <origin xyz="${props.origin.xyz}" rpy="${props.origin.rpy}" />
+      <parent link="${prefix}link2" />
+      <child link="${prefix}link3" />
+      <axis xyz="${props.axis.xyz}" />
+      <xacro:property name="limit" value="${props.limit}" />
+      <limit lower="${limit.lower}" upper="${limit.upper}" effort="${limit.effort}" velocity="${limit.velocity}" />
+    </joint>
+    <xacro:property name="props" value="${joints_props['wrist1']}" />
+    <joint name="${prefix}wrist1" type="revolute">
+      <origin xyz="${props.origin.xyz}" rpy="${props.origin.rpy}" />
+      <parent link="${prefix}link3" />
+      <child link="${prefix}link4" />
+      <axis xyz="${props.axis.xyz}" />
+      <xacro:property name="limit" value="${props.limit}" />
+      <limit lower="${limit.lower}" upper="${limit.upper}" effort="${limit.effort}" velocity="${limit.velocity}" />
+    </joint>
+    <xacro:property name="props" value="${joints_props['wrist2']}" />
+    <joint name="${prefix}wrist2" type="revolute">
+      <origin xyz="${props.origin.xyz}" rpy="${props.origin.rpy}" />
+      <parent link="${prefix}link4" />
+      <child link="${prefix}link5" />
+      <axis xyz="${props.axis.xyz}" />
+      <xacro:property name="limit" value="${props.limit}" />
+      <limit lower="${limit.lower}" upper="${limit.upper}" effort="${limit.effort}" velocity="${limit.velocity}" />
+    </joint>
+    <xacro:property name="props" value="${joints_props['wrist3']}" />
+    <joint name="${prefix}wrist3" type="revolute">
+      <origin xyz="${props.origin.xyz}" rpy="${props.origin.rpy}" />
+      <parent link="${prefix}link5" />
+      <child link="${prefix}link6" />
+      <axis xyz="${props.axis.xyz}" />
+      <xacro:property name="limit" value="${props.limit}" />
+      <limit lower="${limit.lower}" upper="${limit.upper}" effort="${limit.effort}" velocity="${limit.velocity}" />
+    </joint> -->
     <joint name="${prefix}${tcp_name}_joint" type="fixed">
       <origin xyz="${tcp_xyz}" rpy="${tcp_rpy}" />

Commit message: minor changes to launch

File: rbpodo_description/robots/rb10_1300e.urdf.xacro (robot description, xacro)
@@ -4,6 +4,4 @@
   <xacro:include filename="$(find rbpodo_description)/robots/rb_6dof.ros2_control.xacro" />
   <xacro:include filename="$(find rbpodo_description)/robots/rb10_gazebo_control.xacro" />
-  <!-- <xacro:property name="ros2_control_params" value="$(find rbpodo_description)/configs/rb10_controller.yaml" />
-  <xacro:ignition_ros2_control_plugin ros2_control_params:="${ros2_control_params}"> -->
   <xacro:arg name="prefix" default="" />
   <xacro:arg name="robot_ip" default="10.0.2.7"/>
@@ -20,3 +18,5 @@
   <xacro:rb_6dof model_id="rb10_1300e" prefix="$(arg prefix)" tcp_name="tcp" tcp_xyz="0 -0.1153 0" tcp_rpy="0 0 0" />
   <xacro:rb_6dof_ros2_control prefix="$(arg prefix)" robot_ip="$(arg robot_ip)" cb_simulation="$(arg cb_simulation)" use_fake_hardware="$(arg use_fake_hardware)" fake_sensor_commands="$(arg fake_sensor_commands)" torque_constants="${[base_tc, shoulder_tc, elbow_tc, wrist1_tc, wrist2_tc, wrist3_tc]}" />
+  <xacro:property name="new_ros2_control_params" value="$(find rbpodo_description)/configs/rb10_controller.yaml" />
+  <xacro:ignition_ros2_control_plugin ros2_control_params="${new_ros2_control_params}"/>
 </robot>

Commit message: Fixing the dae and stl

File: rbpodo_description/robots/rb10_1300e.urdf.xacro (robot description, xacro)
@@ -4,4 +4,5 @@
   <xacro:include filename="$(find rbpodo_description)/robots/rb_6dof.ros2_control.xacro" />
   <xacro:include filename="$(find rbpodo_description)/robots/rb10_gazebo_control.xacro" />
+  <!-- RB10 Arguments -->
   <xacro:arg name="prefix" default="" />
   <xacro:arg name="robot_ip" default="10.0.2.7"/>

File: rbpodo_description/robots/rb_6dof.xacro (robot description, xacro)
@@ -7,10 +7,10 @@
       <visual>
         <geometry>
-          <mesh filename="package://rbpodo_description/meshes/${model_id}/visual/${name}.dae" />
+          <mesh filename="$(find rbpodo_description)/meshes/${model_id}/visual/${name}.dae" />
         </geometry>
       </visual>
       <collision>
         <geometry>
-          <mesh filename="package://rbpodo_description/meshes/${model_id}/collision/${name}.stl" />
+          <mesh filename="$(find rbpodo_description)/meshes/${model_id}/collision/${name}.stl" />
         </geometry>
       </collision>

Commit message: fix joint_state_broadcaster

File: rbpodo_description/robots/rb10_1300e.urdf.xacro (robot description, xacro)
@@ -18,5 +18,7 @@
   <xacro:property name="wrist3_tc" value="${1}" />
   <xacro:rb_6dof model_id="rb10_1300e" prefix="$(arg prefix)" tcp_name="tcp" tcp_xyz="0 -0.1153 0" tcp_rpy="0 0 0" />
-  <xacro:rb_6dof_ros2_control prefix="$(arg prefix)" robot_ip="$(arg robot_ip)" cb_simulation="$(arg cb_simulation)" use_fake_hardware="$(arg use_fake_hardware)" fake_sensor_commands="$(arg fake_sensor_commands)" torque_constants="${[base_tc, shoulder_tc, elbow_tc, wrist1_tc, wrist2_tc, wrist3_tc]}" />
+  <xacro:rb_6dof_ros2_control prefix="$(arg prefix)" robot_ip="$(arg robot_ip)" cb_simulation="$(arg cb_simulation)"
+                              use_fake_hardware="$(arg use_fake_hardware)" fake_sensor_commands="$(arg fake_sensor_commands)"
+                              torque_constants="${[base_tc, shoulder_tc, elbow_tc, wrist1_tc, wrist2_tc, wrist3_tc]}" />
   <xacro:property name="new_ros2_control_params" value="$(find rbpodo_description)/configs/rb10_controller.yaml" />
   <xacro:ignition_ros2_control_plugin ros2_control_params="${new_ros2_control_params}"/>

File: rbpodo_description/robots/rb_6dof.ros2_control.xacro (robot description, xacro)
@@ -3,15 +3,16 @@
   <xacro:macro name="rb_6dof_ros2_control" params="prefix robot_ip cb_simulation:=true use_fake_hardware:=^|false fake_sensor_commands:=^|false torque_constants:=${[1, 1, 1, 1, 1, 1]}">
     <ros2_control name="RBPodoHardwareInterface" type="system">
-      <hardware>
-        <xacro:if value="${use_fake_hardware}">
+      ]<hardware>
+        <!-- <xacro:if value="${use_fake_hardware}">
           <plugin>mock_components/GenericSystem</plugin>
           <param name="mock_sensor_commands">${fake_sensor_commands}</param>
           <param name="state_following_offset">0.0</param>
-        </xacro:if>
-        <xacro:unless value="${use_fake_hardware}">
+        </xacro:if> -->
+        <plugin>ign_ros2_control/IgnitionSystem</plugin>
+        <!-- <xacro:unless value="${use_fake_hardware}">
           <plugin>rbpodo_hardware/RBPodoHardwareInterface</plugin>
           <param name="cb_simulation">${cb_simulation}</param>
           <param name="robot_ip">${robot_ip}</param>
-        </xacro:unless>
+        </xacro:unless> -->
       </hardware>
       <xacro:macro name="configure_joint" params="joint_name torque_constant:=1">

File: rbpodo_description/robots/rb_6dof.xacro (robot description, xacro)
@@ -57,11 +57,11 @@
     <xacro:link name="${prefix}link6" />
     <link name="${prefix}${tcp_name}" />
-    <xacro:joint name="${prefix}base" prefix="${prefix}"/>
+    <!-- <xacro:joint name="${prefix}base" prefix="${prefix}"/>
     <xacro:joint name="${prefix}shoulder" prefix="${prefix}"/>
     <xacro:joint name="${prefix}elbow" prefix="${prefix}"/>
     <xacro:joint name="${prefix}wrist1" prefix="${prefix}"/>
     <xacro:joint name="${prefix}wrist2" prefix="${prefix}"/>
-    <xacro:joint name="${prefix}wrist3" prefix="${prefix}"/>
-    <!-- <xacro:property name="joints_props_file" value="$(find rbpodo_description)/robots/${model_id}/joint.yaml" />
+    <xacro:joint name="${prefix}wrist3" prefix="${prefix}"/> -->
+    <xacro:property name="joints_props_file" value="$(find rbpodo_description)/robots/${model_id}/joint.yaml" />
     <xacro:property name="joints_props" value="${xacro.load_yaml(joints_props_file)}" />
     <xacro:property name="props" value="${joints_props['base']}" />
@@ -118,5 +118,5 @@
       <xacro:property name="limit" value="${props.limit}" />
       <limit lower="${limit.lower}" upper="${limit.upper}" effort="${limit.effort}" velocity="${limit.velocity}" />
-    </joint> -->
+    </joint>
     <joint name="${prefix}${tcp_name}_joint" type="fixed">
       <origin xyz="${tcp_xyz}" rpy="${tcp_rpy}" />

Commit message: fixed controller and connected to world table

File: rbpodo_description/robots/rb10_1300e.urdf.xacro (robot description, xacro)
@@ -10,4 +10,5 @@
   <xacro:arg name="use_fake_hardware" default="true"/>
   <xacro:arg name="fake_sensor_commands" default="false"/>
+  <xacro:arg name="attach_to" default="world"/>
   <!-- torque_constant = actual_torque_constant * gear_ratio -->
   <xacro:property name="base_tc" value="${1}" />
@@ -17,5 +18,5 @@
   <xacro:property name="wrist2_tc" value="${1}" />
   <xacro:property name="wrist3_tc" value="${1}" />
-  <xacro:rb_6dof model_id="rb10_1300e" prefix="$(arg prefix)" tcp_name="tcp" tcp_xyz="0 -0.1153 0" tcp_rpy="0 0 0" />
+  <xacro:rb_6dof model_id="rb10_1300e" prefix="$(arg prefix)" tcp_name="tcp" tcp_xyz="0 -0.1153 0" tcp_rpy="0 0 0" attach_to='$(arg attach_to)'/>
   <xacro:rb_6dof_ros2_control prefix="$(arg prefix)" robot_ip="$(arg robot_ip)" cb_simulation="$(arg cb_simulation)"
                               use_fake_hardware="$(arg use_fake_hardware)" fake_sensor_commands="$(arg fake_sensor_commands)"

File: rbpodo_description/robots/rb_6dof.ros2_control.xacro (robot description, xacro)
@@ -24,5 +24,5 @@
           <command_interface name="position"/>
           <state_interface name="position"/>
-          <state_interface name="effort"/>
+          <state_interface name="velocity"/>
         </joint>
       </xacro:macro>

File: rbpodo_description/robots/rb_6dof.xacro (robot description, xacro)
@@ -42,11 +42,14 @@
     </joint>
   </xacro:macro>
-  <xacro:macro name="rb_6dof" params="model_id prefix='' tcp_name='tcp' tcp_xyz='0 0 0' tcp_rpy='0 0 0'">
-    <link name="world" />
-    <joint name="${prefix}world_joint" type="fixed">
-      <parent link="world" />
-      <child link="${prefix}link0" />
-      <origin xyz="0 0 0" rpy="0 0 0" />
-    </joint>
+  <xacro:macro name="rb_6dof" params="model_id prefix='' tcp_name='tcp' tcp_xyz='0 0 0' tcp_rpy='0 0 0' attach_to='world'">
+    <!-- add one world link if no 'attach_to' specified  -->
+    <xacro:if value="${attach_to != ''}">
+      <link name="${attach_to}" />
+      <joint name="${prefix}world_joint" type="fixed">
+        <parent link="${attach_to}" />
+        <child link="${prefix}link0" />
+        <origin xyz="0 0 0" rpy="0 0 0" />
+      </joint>
+    </xacro:if>
     <xacro:link name="${prefix}link0" has_inertial="true" />
     <xacro:link name="${prefix}link1" />
@@ -124,4 +127,18 @@
       <child link="${prefix}${tcp_name}" />
     </joint>
+    <gazebo>
+        <plugin filename="ignition-gazebo-pose-publisher-system" name="gz::sim::systems::PosePublisher">
+            <publish_link_pose>false</publish_link_pose>
+            <publish_visual_pose>false</publish_visual_pose>
+            <publish_collision_pose>false</publish_collision_pose>
+            <publish_sensor_pose>false</publish_sensor_pose>
+            <publish_model_pose>true</publish_model_pose>
+            <publish_nested_model_pose>true</publish_nested_model_pose>
+            <use_pose_vector_msg>true</use_pose_vector_msg>
+            <update_frequency>10</update_frequency>
+            <static_publisher>false</static_publisher>
+            <static_update_frequency>10</static_update_frequency>
+        </plugin>
+    </gazebo>
   </xacro:macro>
 </robot>
