Commit message: fixed robot falling over

File: rbpodo_description/robots/rb_6dof.xacro (robot description, xacro)
@@ -76,4 +76,5 @@
       <xacro:property name="limit" value="${props.limit}" />
       <limit lower="${limit.lower}" upper="${limit.upper}" effort="${limit.effort}" velocity="${limit.velocity}" />
+      <dynamics damping="1.0" friction="1.0"/>
     </joint>
     <xacro:property name="props" value="${joints_props['shoulder']}" />
@@ -85,4 +86,5 @@
       <xacro:property name="limit" value="${props.limit}" />
       <limit lower="${limit.lower}" upper="${limit.upper}" effort="${limit.effort}" velocity="${limit.velocity}" />
+      <dynamics damping="1.0" friction="1.0"/>
     </joint>
     <xacro:property name="props" value="${joints_props['elbow']}" />
@@ -94,4 +96,5 @@
       <xacro:property name="limit" value="${props.limit}" />
       <limit lower="${limit.lower}" upper="${limit.upper}" effort="${limit.effort}" velocity="${limit.velocity}" />
+      <dynamics damping="1.0" friction="1.0"/>
     </joint>
     <xacro:property name="props" value="${joints_props['wrist1']}" />
@@ -103,4 +106,5 @@
       <xacro:property name="limit" value="${props.limit}" />
       <limit lower="${limit.lower}" upper="${limit.upper}" effort="${limit.effort}" velocity="${limit.velocity}" />
+      <dynamics damping="1.0" friction="1.0"/>
     </joint>
     <xacro:property name="props" value="${joints_props['wrist2']}" />
@@ -112,4 +116,5 @@
       <xacro:property name="limit" value="${props.limit}" />
       <limit lower="${limit.lower}" upper="${limit.upper}" effort="${limit.effort}" velocity="${limit.velocity}" />
+      <dynamics damping="1.0" friction="1.0"/>
     </joint>
     <xacro:property name="props" value="${joints_props['wrist3']}" />
@@ -121,4 +126,5 @@
       <xacro:property name="limit" value="${props.limit}" />
       <limit lower="${limit.lower}" upper="${limit.upper}" effort="${limit.effort}" velocity="${limit.velocity}" />
+      <dynamics damping="1.0" friction="1.0"/>
     </joint>
     <joint name="${prefix}${tcp_name}_joint" type="fixed">

Commit message: decreased weight and fixed mesh path

File: rbpodo_description/robots/rb_6dof.xacro (robot description, xacro)
@@ -7,10 +7,10 @@
       <visual>
         <geometry>
-          <mesh filename="$(find rbpodo_description)/meshes/${model_id}/visual/${name}.dae" />
+          <mesh filename="file://$(find rbpodo_description)/meshes/${model_id}/visual/${name}.dae" />
         </geometry>
       </visual>
       <collision>
         <geometry>
-          <mesh filename="$(find rbpodo_description)/meshes/${model_id}/collision/${name}.stl" />
+          <mesh filename="file://$(find rbpodo_description)/meshes/${model_id}/collision/${name}.stl" />
         </geometry>
       </collision>
